File: M1648/M1648.kicad_sch (KiCad schematic)
At the start: 14 parts

Commit message: Fix: il segnale A14' adesso è applicato a U6
Parts:
- C1, C2, C3, C4, C5, C6: value (none) -> 100n; footprint (none) -> Capacitor_THT:C_Disc_D3.8mm_W2.6mm_P2.50mm
- J1: value (none) -> Z50Bus; footprint (none) -> Connector_PinHeader_2.54mm:PinHeader_2x25_P2.54mm_Horizontal
- R1: value (none) -> 10k; footprint (none) -> Resistor_THT:R_Axial_DIN0204_L3.6mm_D1.6mm_P7.62mm_Horizontal
- U1: value (none) -> 74LS86; footprint (none) -> Package_DIP:DIP-14_W7.62mm
- U2: value (none) -> 74LS04; footprint (none) -> Package_DIP:DIP-14_W7.62mm
- U3: value (none) -> 74LS139; footprint (none) -> Package_DIP:DIP-16_W7.62mm
- U4: value (none) -> 28C256; footprint (none) -> Package_DIP:DIP-28_W15.24mm
- U5, U6: value (none) -> CY62256-70PC; footprint (none) -> Package_DIP:DIP-28_W15.24mm
Connections:
- net A14': now also U6.1 (A14); no longer U5.1 (A14)
- net GND: now also U5.1 (A14); no longer U6.1 (A14)
