File: M1648/M1648.kicad_pcb (KiCad board)
At the start: 2 copper layers, 99.9 x 64.5 mm, 14 parts, among them J1 Z50Bus, U1 74LS86, U2 74LS04, U3 74LS139, U4 28C256, U5 CY62256-70PC, U6 CY62256-70PC

Commit message: Modificato testo PCB
Other:
- board text added: "AZ80M-MEM1648 v1.0 (20220523) - Memory Board + 16Kb Rom + 48 Kb Ram"
- board text removed: "AZ80M-MEM1648 v1.0 (20220522) - Memory Board + 16Kb Rom + 48 Kb Ram"
Changed lines of the file:
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@@
     (effects (font (size 1.524 1.524) (thickness 0.254)))
   )
-  (gr_text "AZ80M-MEM1648 v1.0 (20220522) - Memory Board +  16Kb Rom + 48 Kb Ram" (at 117.348 67.056) (layer "F.SilkS")
+  (gr_text "AZ80M-MEM1648 v1.0 (20220523) - Memory Board +  16Kb Rom + 48 Kb Ram" (at 117.348 67.056) (layer "F.SilkS")
     (effects (font (size 1 1) (thickness 0.15)) (justify left))
   )
